File: PierogiNixiePSU.kicad_pcb (KiCad board)
At the start: 4 copper layers, 53.1 x 33.3 mm, 19 parts, among them J1 OSTVN02A150, J2 OSTVN02A150, J3 PJ-202A, U1 MAX1771CSAT

Commit message: Added mounting hole
Parts:
- added H2: MountingHole, MountingHole:MountingHole_3.5mm_Pad_Via, F.Cu at (121.8, 101.0)
Routing:
- net GND: vias 45 -> 39
Changed lines of the file:
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@@
     (property "ki_description" "Conn Terminal Block 2 POS 2.54mm Solder ST Thru-Hole 6A")
     (attr through_hole)
-    (fp_text reference "J1" (at -0.53 -4.1) (layer "F.SilkS")
+    (fp_text reference "J1" (at -0.43 -4.1) (layer "F.SilkS")
         (effects (font (size 1.27 1.27) (thickness 0.254)))
     )
@@
     (property "ki_description" "CAP ALUM 0.1UF 20% 200V RADIAL")
     (attr through_hole)
-    (fp_text reference "C4" (at 1.25 -2.1 -90) (layer "F.SilkS")
+    (fp_text reference "C4" (at 0 0 -90) (layer "F.SilkS")
         (effects (font (size 1.27 1.27) (thickness 0.254)))
     )
@@
     (property "ki_description" "Conn Terminal Block 2 POS 2.54mm Solder ST Thru-Hole 6A")
     (attr through_hole)
-    (fp_text reference "J2" (at -0.53 -4.2) (layer "F.SilkS")
+    (fp_text reference "J2" (at -0.43 -4.2) (layer "F.SilkS")
         (effects (font (size 1.27 1.27) (thickness 0.254)))
     )
@@
     (property "Sheetname" "")
     (attr through_hole)
-    (fp_text reference "J3" (at -8.1 3.8 -180) (layer "F.SilkS")
+    (fp_text reference "J3" (at -8.2 4) (layer "F.SilkS")
         (effects (font (size 1.000213 1.000213) (thickness 0.15)))
     )
-    (fp_text value "PJ-202A" (at -0.20519 5.77966 90) (layer "F.Fab")
+    (fp_text value "PJ-202A" (at -0.20519 5.77966 -90) (layer "F.Fab")
         (effects (font (size 1.000803 1.000803) (thickness 0.15)))
     )
@@
     )
   )
+  (footprint "MountingHole:MountingHole_3.5mm_Pad_Via" (layer "F.Cu")
+    (at 121.843845 101.043845)
+    (descr "Mounting Hole 3.5mm")
+    (tags "mounting hole 3.5mm")
+    (property "Sheetfile" "PierogiNixiePSU.kicad_sch")
+    (property "Sheetname" "")
+    (property "ki_description" "Mounting Hole without connection")
+    (property "ki_keywords" "mounting hole")
+    (attr exclude_from_pos_files)
+    (fp_text reference "H2" (at 0 -4.5) (layer "F.SilkS") hide
+        (effects (font (size 1 1) (thickness 0.15)))
+    )
+    (fp_text value "MountingHole" (at 0 4.5) (layer "F.Fab") hide
+        (effects (font (size 1 1) (thickness 0.15)))
+    )
+    (fp_text user "${REFERENCE}" (at 0 0) (layer "F.Fab")
+        (effects (font (size 1 1) (thickness 0.15)))
+    )
+    (fp_circle (center 0 0) (end 3.5 0)
+      (stroke (width 0.15) (type solid)) (fill none) (layer "Cmts.User"))
+    (fp_circle (center 0 0) (end 3.75 0)
+      (stroke (width 0.05) (type solid)) (fill none) (layer "F.CrtYd"))
+    (pad "1" thru_hole circle (at -2.625 0) (size 0.8 0.8) (drill 0.5) (layers "*.Cu" "*.Mask"))
+    (pad "1" thru_hole circle (at -1.856155 -1.856155) (size 0.8 0.8) (drill 0.5) (layers "*.Cu" "*.Mask"))
+    (pad "1" thru_hole circle (at -1.856155 1.856155) (size 0.8 0.8) (drill 0.5) (layers "*.Cu" "*.Mask"))
+    (pad "1" thru_hole circle (at 0 -2.625) (size 0.8 0.8) (drill 0.5) (layers "*.Cu" "*.Mask"))
+    (pad "1" thru_hole circle (at 0 0) (size 7 7) (drill 3.5) (layers "*.Cu" "*.Mask"))
+    (pad "1" thru_hole circle (at 0 2.625) (size 0.8 0.8) (drill 0.5) (layers "*.Cu" "*.Mask"))
+    (pad "1" thru_hole circle (at 1.856155 -1.856155) (size 0.8 0.8) (drill 0.5) (layers "*.Cu" "*.Mask"))
+    (pad "1" thru_hole circle (at 1.856155 1.856155) (size 0.8 0.8) (drill 0.5) (layers "*.Cu" "*.Mask"))
+    (pad "1" thru_hole circle (at 2.625 0) (size 0.8 0.8) (drill 0.5) (layers "*.Cu" "*.Mask"))
+  )
   (footprint "footprints:HVSMALL" (layer "B.Cu")
     (at 147.81055 103.73115 180)
@@
   (segment (start 148.3 113.7) (end 148.3 117.45) (width 0.508) (layer "F.Cu") (net 1))
   (segment (start 129.2 103.8) (end 129.3 103.7) (width 0.508) (layer "F.Cu") (net 1))
-  (via (at 118.1 106.3) (size 1) (drill 0.6) (layers "F.Cu" "B.Cu") (free) (net 1))
+  (via (at 126.9 101.1) (size 1) (drill 0.6) (layers "F.Cu" "B.Cu") (free) (net 1))
   (via (at 142.7 117.6) (size 1) (drill 0.6) (layers "F.Cu" "B.Cu") (free) (net 1))
-  (via (at 121.3 97.5) (size 1) (drill 0.6) (layers "F.Cu" "B.Cu") (free) (net 1))
-  (via (at 124.4 100.9) (size 1) (drill 0.6) (layers "F.Cu" "B.Cu") (free) (net 1))
+  (via (at 125.9 107.3) (size 1) (drill 0.6) (layers "F.Cu" "B.Cu") (free) (net 1))
   (via (at 160.7 113.4) (size 1) (drill 0.6) (layers "F.Cu" "B.Cu") (free) (net 1))
   (via (at 152 111.4) (size 1) (drill 0.6) (layers "F.Cu" "B.Cu") (free) (net 1))
+  (via (at 122 94.5) (size 1) (drill 0.6) (layers "F.Cu" "B.Cu") (free) (net 1))
   (via (at 137.4 114.1) (size 1) (drill 0.6) (layers "F.Cu" "B.Cu") (free) (net 1))
-  (via (at 123.596113 89.890947) (size 1) (drill 0.6) (layers "F.Cu" "B.Cu") (free) (net 1))
-  (via (at 118.2 97) (size 1) (drill 0.6) (layers "F.Cu" "B.Cu") (free) (net 1))
   (via (at 167.6 96) (size 1) (drill 0.6) (layers "F.Cu" "B.Cu") (free) (net 1))
-  (via (at 125.2 98.4) (size 1) (drill 0.6) (layers "F.Cu" "B.Cu") (free) (net 1))
   (via (at 166.5 111.6) (size 1) (drill 0.6) (layers "F.Cu" "B.Cu") (free) (net 1))
-  (via (at 124.9 103.7) (size 1) (drill 0.6) (layers "F.Cu" "B.Cu") (free) (net 1))
   (via (at 166.9 101.1) (size 1) (drill 0.6) (layers "F.Cu" "B.Cu") (free) (net 1))
-  (via (at 121 100.7) (size 1) (drill 0.6) (layers "F.Cu" "B.Cu") (free) (net 1))
+  (via (at 128.9 111.8) (size 1) (drill 0.6) (layers "F.Cu" "B.Cu") (free) (net 1))
   (via (at 154.7 111.9) (size 1) (drill 0.6) (layers "F.Cu" "B.Cu") (free) (net 1))
   (via (at 142 108.5) (size 1) (drill 0.6) (layers "F.Cu" "B.Cu") (free) (net 1))
   (via (at 164.7 94) (size 1) (drill 0.6) (layers "F.Cu" "B.Cu") (free) (net 1))
-  (via (at 124.7 95.1) (size 1) (drill 0.6) (layers "F.Cu" "B.Cu") (free) (net 1))
   (via (at 156.9 106.5) (size 1) (drill 0.6) (layers "F.Cu" "B.Cu") (free) (net 1))
-  (via (at 124.8 92.1) (size 1) (drill 0.6) (layers "F.Cu" "B.Cu") (free) (net 1))
+  (via (at 118.8 94.7) (size 1) (drill 0.6) (layers "F.Cu" "B.Cu") (free) (net 1))
+  (via (at 118.6 107.9) (size 1) (drill 0.6) (layers "F.Cu" "B.Cu") (free) (net 1))
   (via (at 139.9 95.3) (size 1) (drill 0.6) (layers "F.Cu" "B.Cu") (free) (net 1))
-  (via (at 118.1 93) (size 1) (drill 0.6) (layers "F.Cu" "B.Cu") (free) (net 1))
+  (via (at 121.9 90.5) (size 1) (drill 0.6) (layers "F.Cu" "B.Cu") (free) (net 1))
   (via (at 141 102.5) (size 1) (drill 0.6) (layers "F.Cu" "B.Cu") (free) (net 1))
-  (via (at 120.3 90.1) (size 1) (drill 0.6) (layers "F.Cu" "B.Cu") (free) (net 1))
   (via (at 157.7 103.4) (size 1) (drill 0.6) (layers "F.Cu" "B.Cu") (free) (net 1))
+  (via (at 122.7 107.7) (size 1) (drill 0.6) (layers "F.Cu" "B.Cu") (free) (net 1))
   (via (at 154.3 103) (size 1) (drill 0.6) (layers "F.Cu" "B.Cu") (free) (net 1))
   (via (at 143.8 113.5) (size 1) (drill 0.6) (layers "F.Cu" "B.Cu") (free) (net 1))
   (via (at 156.9 101.2) (size 1) (drill 0.6) (layers "F.Cu" "B.Cu") (free) (net 1))
-  (via (at 120.2 107.5) (size 1) (drill 0.6) (layers "F.Cu" "B.Cu") (free) (net 1))
   (via (at 154.5 99.2) (size 1) (drill 0.6) (layers "F.Cu" "B.Cu") (free) (net 1))
-  (via (at 120.7 93.4) (size 1) (drill 0.6) (layers "F.Cu" "B.Cu") (free) (net 1))
+  (via (at 126.2 94.6) (size 1) (drill 0.6) (layers "F.Cu" "B.Cu") (free) (net 1))
+  (via (at 125.9 90.8) (size 1) (drill 0.6) (layers "F.Cu" "B.Cu") (free) (net 1))
   (via (at 148.7 111.2) (size 1) (drill 0.6) (layers "F.Cu" "B.Cu") (free) (net 1))
   (via (at 139.3 105.6) (size 1) (drill 0.6) (layers "F.Cu" "B.Cu") (free) (net 1))
-  (via (at 123.6 106.5) (size 1) (drill 0.6) (layers "F.Cu" "B.Cu") (free) (net 1))
   (via (at 147.3 106.2) (size 1) (drill 0.6) (layers "F.Cu" "B.Cu") (free) (net 1))
   (via (at 148.3 113.7) (size 1) (drill 0.6) (layers "F.Cu" "B.Cu") (free) (net 1))
@@
   (via (at 136.8 103.6) (size 1) (drill 0.6) (layers "F.Cu" "B.Cu") (free) (net 1))
   (via (at 154.7 90.6) (size 1) (drill 0.6) (layers "F.Cu" "B.Cu") (free) (net 1))
-  (via (at 120.3 103.9) (size 1) (drill 0.6) (layers "F.Cu" "B.Cu") (free) (net 1))
   (via (at 129.3 103.7) (size 1) (drill 0.6) (layers "F.Cu" "B.Cu") (free) (net 1))
   (via (at 138 119.7) (size 1) (drill 0.6) (layers "F.Cu" "B.Cu") (free) (net 1))
   (via (at 167.7 89.9) (size 1) (drill 0.6) (layers "F.Cu" "B.Cu") (free) (net 1))
-  (via (at 118.1 101.6) (size 1) (drill 0.6) (layers "F.Cu" "B.Cu") (free) (net 1))
+  (via (at 118.7 91.4) (size 1) (drill 0.6) (layers "F.Cu" "B.Cu") (free) (net 1))
   (segment (start 145.375 119.605) (end 148.045 119.605) (width 0.8128) (layer "F.Cu") (net 2))
   (segment (start 148.045 119.605) (end 148.3 119.35) (width 0.8128) (layer "F.Cu") (net 2))

Commit message: Updated schematic and fixed thickness of GND traces
Changed lines of the file:
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@@
     (property "ki_description" "CAP ALUM 0.1UF 20% 200V RADIAL")
     (attr through_hole)
-    (fp_text reference "C4" (at 0 0 -90) (layer "F.SilkS")
+    (fp_text reference "C4" (at 1.55 -2.2 -90) (layer "F.SilkS")
         (effects (font (size 1.27 1.27) (thickness 0.254)))
     )
@@
     (effects (font (size 0.7 0.7) (thickness 0.1)) (justify left bottom))
   )
-  (segment (start 138.095 119.605) (end 138 119.7) (width 0.508) (layer "F.Cu") (net 1))
-  (segment (start 140.425 119.605) (end 138.095 119.605) (width 0.508) (layer "F.Cu") (net 1))
   (segment (start 142.3 116.3) (end 143.9 116.3) (width 0.508) (layer "F.Cu") (net 1))
   (segment (start 152.1 111.5) (end 152 111.4) (width 0.508) (layer "F.Cu") (net 1))
   (segment (start 142.7 117.6) (end 143.3 117.6) (width 0.508) (layer "F.Cu") (net 1))
-  (segment (start 139.3 109.3) (end 139.3 105.6) (width 0.508) (layer "F.Cu") (net 1))
+  (segment (start 139.3 109.3) (end 139.3 105.6) (width 1) (layer "F.Cu") (net 1))
   (segment (start 144.665 117.065) (end 145.375 117.065) (width 0.508) (layer "F.Cu") (net 1))
-  (segment (start 129.2 107.45) (end 129.2 103.8) (width 0.508) (layer "F.Cu") (net 1))
   (segment (start 156.878 106.478) (end 154.5 106.478) (width 0.508) (layer "F.Cu") (net 1))
+  (segment (start 138.095 119.605) (end 140.425 119.605) (width 0.8128) (layer "F.Cu") (net 1))
   (segment (start 143.3 117.6) (end 144.035 118.335) (width 0.508) (layer "F.Cu") (net 1))
   (segment (start 143.9 116.3) (end 144.665 117.065) (width 0.508) (layer "F.Cu") (net 1))
@@
   (segment (start 156.9 106.5) (end 156.878 106.478) (width 0.508) (layer "F.Cu") (net 1))
   (segment (start 144.035 118.335) (end 145.375 118.335) (width 0.508) (layer "F.Cu") (net 1))
+  (segment (start 138 119.7) (end 138.095 119.605) (width 0.8128) (layer "F.Cu") (net 1))
   (segment (start 156.9 99.25) (end 156.9 101.2) (width 0.508) (layer "F.Cu") (net 1))
-  (segment (start 148.3 113.7) (end 148.3 117.45) (width 0.508) (layer "F.Cu") (net 1))
-  (segment (start 129.2 103.8) (end 129.3 103.7) (width 0.508) (layer "F.Cu") (net 1))
+  (segment (start 129.2 103.8) (end 129.2 107.45) (width 0.8128) (layer "F.Cu") (net 1))
+  (segment (start 148.3 113.7) (end 148.3 117.45) (width 0.8128) (layer "F.Cu") (net 1))
   (via (at 126.9 101.1) (size 1) (drill 0.6) (layers "F.Cu" "B.Cu") (free) (net 1))
   (via (at 142.7 117.6) (size 1) (drill 0.6) (layers "F.Cu" "B.Cu") (free) (net 1))
@@
   (via (at 136.8 103.6) (size 1) (drill 0.6) (layers "F.Cu" "B.Cu") (free) (net 1))
   (via (at 154.7 90.6) (size 1) (drill 0.6) (layers "F.Cu" "B.Cu") (free) (net 1))
-  (via (at 129.3 103.7) (size 1) (drill 0.6) (layers "F.Cu" "B.Cu") (free) (net 1))
+  (via (at 129.2 103.8) (size 1) (drill 0.6) (layers "F.Cu" "B.Cu") (free) (net 1))
   (via (at 138 119.7) (size 1) (drill 0.6) (layers "F.Cu" "B.Cu") (free) (net 1))
   (via (at 167.7 89.9) (size 1) (drill 0.6) (layers "F.Cu" "B.Cu") (free) (net 1))
