File: V1.1/PierogiNixiePSU.kicad_sch (KiCad schematic)
At the start: 19 parts, among them J1 OSTVN02A150, J2 OSTVN02A150, J4 Barrel_Jack, Q1 IRF740STRLPBF, U1 MAX1771CSAT

Commit message: dded Gerbers
Parts:
- renumbered J4 to J3
Changed lines of the file:
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@@
   (symbol (lib_id "Connector:Barrel_Jack") (at 57.15 58.42 0) (unit 1)
     (in_bom yes) (on_board yes) (dnp no)
-    (property "Reference" "J4" (at 57.15 53.34 0)
+    (property "Reference" "J3" (at 57.15 53.34 0)
       (effects (font (size 1.27 1.27)))
     )
@@
       (project "PierogiNixiePSU"
         (path "/aae08d1b-aae6-480a-b174-6c54c1927943"
-          (reference "J4") (unit 1)
+          (reference "J3") (unit 1)
         )
       )
